File: Peripherals Board/Peripherals Board (new).kicad_pcb (KiCad board)
At the start: 2 copper layers, 50.8 x 40.6 mm, 16 parts, among them J1 Conn_01x02_Pin, J2 Conn_01x05_Pin, J4 Conn_02x11_Counter_Clockwise, U1 Teensy4.0, U2 SN65HVD230, U3 74AHC125

Commit message: minor changes
Parts:
- moved H1 0.90 mm to (217.8, 48.9)
- moved H3 0.90 mm to (173.4, 48.9)
- moved H2 0.90 mm to (217.8, 83.2)
- moved H4 0.90 mm to (173.4, 83.2)
Routing:
- net +5V: track 85.6 -> 84.9 mm
