File: Power Board/Power Board.kicad_sch (KiCad schematic)
At the start: 8 parts, among them IC1 LTC4151IMS#PBF, U1 BQ34Z100PW

Commit message: working on power board
Parts:
- removed R4: R, symbol Device:R
- removed U1: BQ34Z100PW, PW14_TEX, symbol BQ34Z100PW:BQ34Z100PW
- added C10: 10 uF, symbol Device:C
- added C11, C16, C3, C5, C7, C8, C9: 10nF, symbol Device:C
- added C12, C13, C14, C15, C17, C4, C6: 100 nF, symbol Device:C
- added C18, C22: 0.1 uF, symbol Device:C
- added C19, C20, C21, C23: 1 uF, symbol Device:C
- added D7 (x8): D_Zener, Diode_SMD:D_SOD-123, symbol Device:D_Zener
- added F1 (x8): Fuse, SOCMonitor:FUSE_3568, symbol Device:Fuse
- added J8 (x9): Conn_01x02, SOCMonitor:MOLEX_768290102, symbol Connector_Generic:Conn_01x02
- added K1: Relay_DPST-NO, symbol Relay:Relay_DPST-NO
- added Q10, Q11, Q12, Q13, Q14, Q15, Q16, Q17, Q18, Q19, Q20, Q21, Q22, Q9: Q_NMOS_GDS, symbol Device:Q_NMOS_GDS
- added Q9 (x8): Q_PMOS_GDS, Package_TO_SOT_SMD:TO-252-2, symbol Device:Q_PMOS_GDS
- added R13, R16, R19, R20, R23, R24, R31: 10, symbol Device:R
- added R14, R17, R21, R25, R26, R27, R32: R, symbol Device:R
- added R15, R18, R22, R28, R29, R30, R33: 100, symbol Device:R
- added R34: 20k, symbol Device:R
- added R35: 10k, symbol Device:R
- added R8 (x8): 100k, Resistor_SMD:R_0805_2012Metric_Pad1.20x1.40mm_HandSolder, symbol Device:R
- added TP11 (x9): TestPoint, TestPoint:TestPoint_Pad_1.5x1.5mm, symbol Connector:TestPoint
- added U1: ADR395, Package_TO_SOT_SMD:SOT-23-5, symbol ADR395:ADR395
- added U10, U2, U3, U4, U5, U6, U7: LTC4372, symbol LTC4372:LTC4372
- added U11: ACS770xCB-200U-PFF, Sensor_Current:Allegro_CB_PFF, symbol Sensor_Current:ACS770xCB-200U-PFF
- added U8: ADC128S052CIMT, ADC128S052CIMT:SOP65P640X120-16N, symbol ADC128S052CIMT:ADC128S052CIMT
- added U9: L7805, symbol Regulator_Linear:L7805
- C1: value 1 μF -> 22 nF
- C2: value 0.1 μF -> 22 nF
- R1: value 0.02 -> 0.04
- R2, R3: value R -> 100
Connections:
- net BAT- is gone; now on an unnamed net: R2.2
- net V_ADin is gone; now on net GND: IC1.5 (ADIN)
- net GND: now also C10.2, C11.2, C16.2, C18.2, C19.2, C20.2, C21.2, C22.2, C23.2, C3.2, C5.2, C7.2, C8.2, C9.2, J8.1 (Pin_1), J8.1 (Pin_1), J8.1 (Pin_1), J8.1 (Pin_1), J8.1 (Pin_1), J8.1 (Pin_1), J8.1 (Pin_1), J8.1 (Pin_1), K1.A1, R15.2, R18.2, R22.2, R28.2, R29.2, R30.2, R33.2, R35.2, R8.2, R8.2, R8.2, R8.2, R8.2, R8.2, R8.2, R8.2, U1. (VOUT_S), U11.2 (GND), U8.12 (DGND), U8.3 (AGND), U9.2 (GND)
- net at R3.2: now also C2.1, U8.4 (IN0)
- net at C1.1: now also U8.5 (IN1)
- net BAT+ renamed 12V_AMP_SENSE
- net 12V_AMP_SENSE: now also U11.3 (VIOUT)
- net PACK-: no longer names the net of R2.1
- net PACK-: now also R34.2, R35.1
- net SCL renamed 24V_MONITOR_SCL
- net SDA renamed 24V_MONITOR_SDA
- net V_IN renamed 24V_PRESENSE
- net 24V_PRESENSE: now also K1.14
- net V_OUT renamed 24V_UNREGULATED
- new net: D7.2 (A), Q9.1 (G), R8.1 (x8)
- new net: F1.2, Q9.2 (D) (x8)
- new net: Q11.1 (G), R16.1, R17.1, U3. (SOURCE)
- new net: Q11.3 (S), Q12.3 (S), U3. (SOURCE)
- new net: C6.1, R18.1, U3. (SOURCE)
- new net: C6.2, U3. (SOURCE)
- new net: C3.1, R14.2
- new net: C12.1, R22.1, U10. (SOURCE)
- new net: C12.2, U10. (SOURCE)
- new net: F1.1, J8.2 (Pin_2) (x8)
- new net: Q21.1 (G), R31.1, R32.1, U7. (SOURCE)
- new net: Q21.3 (S), Q22.3 (S), U7. (SOURCE)
- new net: Q15.1 (G), R23.1, R26.1, U5. (SOURCE)
- new net: C8.1, R26.2
- new net: C4.1, R15.1, U2. (SOURCE)
- new net: C4.2, U2. (SOURCE)
- new net: C14.1, R29.1, U5. (SOURCE)
- new net: Q15.3 (S), Q16.3 (S), U5. (SOURCE)
- new net: C14.2, U5. (SOURCE)
- new net: Q12.1 (G), R16.2
- new net: Q9.1 (G), R13.1, R14.1, U2. (SOURCE)
- new net: Q10.3 (S), Q9.3 (S), U2. (SOURCE)
- new net: Q10.1 (G), R13.2
- new net: Q19.1 (G), R24.1, R27.1, U6. (SOURCE)
- new net: C9.1, R27.2
- new net: Q18.1 (G), R20.1, R21.1, U10. (SOURCE)
- new net: Q17.3 (S), Q18.3 (S), U10. (SOURCE)
- new net: C15.1, R30.1, U6. (SOURCE)
- new net: C15.2, U6. (SOURCE)
- new net: Q17.1 (G), R20.2
- new net: C17.1, R33.1, U7. (SOURCE)
- new net: C17.2, U7. (SOURCE)
- new net: C13.1, R28.1, U4. (SOURCE)
- new net: C13.2, U4. (SOURCE)
- new net: Q13.1 (G), R19.1, R25.1, U4. (SOURCE)
- new net: Q13.3 (S), Q14.3 (S), U4. (SOURCE)
- new net: C5.1, R17.2
- new net: Q19.3 (S), Q20.3 (S), U6. (SOURCE)
- new net: Q20.1 (G), R24.2
- new net: Q16.1 (G), R23.2
- new net: C16.1, R32.2
- new net: Q22.1 (G), R31.2
- new net: J8.2 (Pin_2), K1.A2
- new net: C7.1, R25.2
- new net: C11.1, R21.2
- new net: Q14.1 (G), R19.2
- new net +5V: C22.1, C23.1, U11.1 (VCC)
- new net 12V_PRESENSE: Q11.2 (D), Q13.2 (D), Q15.2 (D), Q18.2 (D), Q19.2 (D), Q21.2 (D), Q9.2 (D), R34.1, U10. (SOURCE), U11.4 (IP+), U2. (SOURCE), U3. (SOURCE), U4. (SOURCE), U5. (SOURCE), U6. (SOURCE), U7. (SOURCE)
- new net 12V_PSO: C10.1, TP11.1
- new net 12V_UNREGULATED: U1. (VOUT_S), U11.5 (IP-)
- new net 24V_PSO: D7.1 (K), K1.13, Q9.3 (S), TP11.1, U9.1 (IN)
- new net 5V_REF: C18.1, C19.1, C20.1, C21.1, U1. (VOUT_S), U8.13 (VD), U8.2 (VA)
- new net 5V_REG_SD: J8.1 (Pin_1), K1.24, U9.3 (OUT)
- new net ADC_1_CS: U8.1 (~{CS})
- new net ADC_1_DIN: U8.14 (DIN)
- new net ADC_1_DOUT: U8.15 (DOUT)
- new net ADC_1_SCLK: U8.16 (SCLK)
- new net BATT_IN_12_1: D7.1 (K), Q17.2 (D), Q9.3 (S), TP11.1, U10. (SOURCE)
- new net BATT_IN_12_2: D7.1 (K), Q10.2 (D), Q9.3 (S), TP11.1, U2. (SOURCE)
- new net BATT_IN_12_3: D7.1 (K), Q12.2 (D), Q9.3 (S), TP11.1, U3. (SOURCE)
- new net BATT_IN_12_4: D7.1 (K), Q14.2 (D), Q9.3 (S), TP11.1, U4. (SOURCE)
- new net BATT_IN_12_5: D7.1 (K), Q16.2 (D), Q9.3 (S), TP11.1, U5. (SOURCE)
- new net BATT_IN_12_6: D7.1 (K), Q20.2 (D), Q9.3 (S), TP11.1, U6. (SOURCE)
- new net BATT_IN_12_7: D7.1 (K), Q22.2 (D), Q9.3 (S), TP11.1, U7. (SOURCE)
- new net SHDN: K1.23, U10. (SOURCE), U2. (SOURCE), U3. (SOURCE), U4. (SOURCE), U5. (SOURCE), U6. (SOURCE), U7. (SOURCE)
Other:
- note added: "Battery Connectors"
- note added: "Battery Monitors"
- note added: "Parallel, Shutdown Circuitry"
- note removed: "1"
- note removed: "Power Board"
- note removed: "University Rover Challenge Princeton University"
- company: (none) -> Princeton University Rover Team
- title: (none) -> Power Board
- moved on the sheet: IC1, R1

Commit message: working on power board
Parts:
- added C26: 0.1 uF, symbol Device:C
- added C27, C28, C29: 1 uF, symbol Device:C
- added J8 (x8): Conn_01x02, SOCMonitor:MOLEX_768290102, symbol Connector_Generic:Conn_01x02
- added R36, R37, R38, R39, R4, R40, R41, R42: R, symbol Device:R
- added U12: ADC128S052CIMT, ADC128S052CIMT:SOP65P640X120-16N, symbol ADC128S052CIMT:ADC128S052CIMT
- added U13: ADR395, Package_TO_SOT_SMD:SOT-23-5, symbol ADR395:ADR395
Connections:
- net 12V_UNREGULATED: now also U13. (VOUT_S)
- net ADC_1_CS: now also U12.1 (~{CS})
- net ADC_1_DIN: now also U12.14 (DIN)
- net ADC_1_DOUT: now also U12.15 (DOUT)
- net ADC_1_SCLK: now also U12.16 (SCLK)
- net GND: now also C26.2, C27.2, C28.2, C29.2, R36.2, R37.2, R38.2, R39.2, R4.2, R40.2, R41.2, R42.2, U12.12 (DGND), U12.3 (AGND), U13. (VOUT_S)
- net 5V_REF renamed 5V_REF_1
- new net 5V_REF_2: C26.1, C27.1, C28.1, C29.1, U12.13 (VD), U12.2 (VA), U13. (VOUT_S)
- new net 5V_REF_V2: J8.2 (Pin_2), J8.2 (Pin_2), J8.2 (Pin_2), J8.2 (Pin_2), J8.2 (Pin_2), J8.2 (Pin_2), J8.2 (Pin_2), J8.2 (Pin_2)
- new net THERM_1: J8.1 (Pin_1), R4.1, U12.4 (IN0)
- new net THERM_2: J8.1 (Pin_1), R36.1, U12.5 (IN1)
- new net THERM_3: J8.1 (Pin_1), R37.1, U12.6 (IN2)
- new net THERM_4: J8.1 (Pin_1), R38.1, U12.7 (IN3)
- new net THERM_5: J8.1 (Pin_1), R39.1, U12.8 (IN4)
- new net THERM_6: J8.1 (Pin_1), R40.1, U12.9 (IN5)
- new net THERM_7: J8.1 (Pin_1), R41.1, U12.10 (IN6)
- new net THERM_8: J8.1 (Pin_1), R42.1, U12.11 (IN7)
Other:
- note added: "Battery Monitor"
- note added: "Battery Monitor ADC"
- note added: "Thermistor"
- note added: "Thermistor ADC"
- note removed: "Battery Monitors"
- moved on the sheet: C1, C18, C19, C2, C20, C21, C22, C23, IC1, R1, R2, R3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

Commit message: power board update
Parts:
- removed J8: Conn_01x02, SOCMonitor:MOLEX_768290102, symbol Connector_Generic:Conn_01x02
- removed K1: Relay_DPST-NO, symbol Relay:Relay_DPST-NO
- removed U1, U13: ADR395, Package_TO_SOT_SMD:SOT-23-5, symbol ADR395:ADR395
- removed U10, U2, U3, U4, U5, U6, U7: LTC4372, symbol LTC4372:LTC4372
- removed U9: L7805, symbol Regulator_Linear:L7805
- added C24, C25: 330 uF, symbol Device:C
- added D10, D9: D_Zener, Diode_SMD:D_SMB, symbol Device:D_Zener
- added J19, J20: Conn_01x04, symbol Connector_Generic:Conn_01x04
- added J_JETSON1, J_PDB1, J_PERIPHERAL1, J_PIX1, J_PIX2, J_ROCKET1, J_SERVO1: Conn_01x02, symbol Connector_Generic:Conn_01x02
- added PS1: THN_10-4815WIR, THN_10_4815WIR:CONV_THN_10-4815WIR, symbol THN_10-4815WIR:THN_10-4815WIR
- added PS2: JTK3024S05, JTK3024S05:JTK3024S05, symbol JTK3024S05:JTK3024S05
- added SW1: SW_Push_DPDT, symbol Switch:SW_Push_DPDT
- added U1: TLV70033_SOT23-5, Package_TO_SOT_SMD:SOT-23-5, symbol Regulator_Linear:TLV70033_SOT23-5
- added U2, U3, U4, U5, U6, U7, U9: LTC4372CDD-PBF, footprints:05-08-1698_ADI, symbol LTC4372:LTC4372CDD-PBF
- C20, C21: value 1 uF -> 0.1 uF
- C28, C29: value 1 uF -> C
- F1: footprint SOCMonitor:FUSE_3568 -> 0498060:Fuse_0498060M
- F2, F3, F4, F5, F6, F7, F8: renamed from F1; footprint SOCMonitor:FUSE_3568 -> 0498060:Fuse_0498060M
- IC1: footprint SOP50P490X110-10N -> LTC4151:MSOP-10_MS_LIT
- J1, J2, J3, J4, J5, J6, J7: renamed from J8; footprint SOCMonitor:MOLEX_768290102 -> Connector_AMASS:AMASS_XT60PW-F_1x02_P7.20mm_Horizontal
- J10, J11, J12, J13, J14, J15, J16, J17: renamed from J8; footprint SOCMonitor:MOLEX_768290102 -> Connector_Molex:Molex_KK-254_AE-6410-02A_1x02_P2.54mm_Vertical
- J8: footprint SOCMonitor:MOLEX_768290102 -> Connector_AMASS:AMASS_XT60PW-F_1x02_P7.20mm_Horizontal
- Q1, Q2, Q3, Q4, Q5, Q6, Q7, Q8: renamed from Q9; footprint Package_TO_SOT_SMD:TO-252-2 -> Package_SO:PowerPAK_SO-8_Single
- Q10, Q11, Q12, Q13, Q14, Q15, Q16, Q17, Q18, Q19, Q20, Q21, Q22, Q9: footprint (none) -> Package_TO_SOT_SMD:TDSON-8-1
- U12, U8: footprint ADC128S052CIMT:SOP65P640X120-16N -> ADC128S052CIMT_NOPB:SOP65P640X120-16N
- renumbered D7 to D1, D7 to D2, D7 to D3, D7 to D4, D7 to D5, D7 to D6, D7 to D8, R8 to R10, R8 to R11, R8 to R12, R8 to R5, R8 to R6, R8 to R7, R8 to R9, TP11 to TP1, TP11 to TP2, TP11 to TP3, TP11 to TP4, TP11 to TP5, TP11 to TP6, TP11 to TP7, TP11 to TP8, TP11 to TP9
Connections:
- net 5V_REF_V2 is gone; now on net 5V_REGULATED: J10.2 (Pin_2), J11.2 (Pin_2), J12.2 (Pin_2), J13.2 (Pin_2), J14.2 (Pin_2), J15.2 (Pin_2), J16.2 (Pin_2), J17.2 (Pin_2)
- net 12V_PRESENSE: now also U2.1 (OUT), U3.1 (OUT), U4.1 (OUT), U6.1 (OUT), U7.1 (OUT), U9.1 (OUT)
- net 12V_UNREGULATED: now also J_JETSON1.2 (Pin_2), J_PDB1.2 (Pin_2), J_PIX1.2 (Pin_2), J_PIX2.2 (Pin_2), J_SERVO1.2 (Pin_2)
- net 24V_PSO: now also SW1.5 (B)
- net 24V_UNREGULATED: now also C24.2, C25.1, D10.1 (K), D9.1 (K), PS1.1 (+VIN(VCC)), PS2.1 (+VIN), SW1.4 (A)
- net 5V_REG_SD: now also SW1.3 (C)
- net ADC_1_CS: now also J20.1 (Pin_1); no longer U12.1 (~{CS})
- net ADC_1_DIN: now also J20.3 (Pin_3); no longer U12.14 (DIN)
- net ADC_1_DOUT: now also J20.4 (Pin_4); no longer U12.15 (DOUT)
- net ADC_1_SCLK: now also J20.2 (Pin_2); no longer U12.16 (SCLK)
- net BATT_IN_12_1: now also U9.4 (IN)
- net BATT_IN_12_2: now also U2.4 (IN)
- net BATT_IN_12_3: now also U3.4 (IN)
- net BATT_IN_12_4: now also U4.4 (IN)
- net BATT_IN_12_5: now also U5.4 (IN)
- net BATT_IN_12_6: now also U6.4 (IN)
- net BATT_IN_12_7: now also U7.4 (IN)
- net GND: now also C24.1, C25.2, D10.2 (A), D9.2 (A), J_JETSON1.1 (Pin_1), J_PDB1.1 (Pin_1), J_PIX1.1 (Pin_1), J_PIX2.1 (Pin_1), J_SERVO1.1 (Pin_1), PS1.2 (-VIN(GND)), PS1.6 (-VOUT), PS2.2 (-VIN), PS2.4 (+VOUT), SW1.1 (A), U1.2 (GND); no longer C18.2, C19.2, C26.2, C27.2, U12.12 (DGND), U8.12 (DGND)
- net SHDN: now also SW1.2 (B), U2.8 (SHDN), U3.8 (SHDN), U4.8 (SHDN), U5.8 (SHDN), U6.8 (SHDN), U7.8 (SHDN), U9.8 (SHDN)
- net at Q11.1 (G), R16.1, R17.1: now also U3.2 (GATE)
- net at Q11.3 (S), Q12.3 (S): now also U3.3 (SOURCE)
- net at C6.1, R18.1: now also U3.6 (GND)
- net at C6.2: now also U3.5 (INTVCC)
- net at C12.1, R22.1: now also U9.6 (GND)
- net at C12.2: now also U9.5 (INTVCC)
- net at Q21.1 (G), R31.1, R32.1: now also U7.2 (GATE)
- net at Q21.3 (S), Q22.3 (S): now also U7.3 (SOURCE)
- net at C4.1, R15.1: now also U2.6 (GND)
- net at C4.2: now also U2.5 (INTVCC)
- net at C14.1, R29.1: now also U5.6 (GND)
- net at C14.2: now also U5.5 (INTVCC)
- net at Q9.1 (G), R13.1, R14.1: now also U2.2 (GATE)
- net at Q10.3 (S), Q9.3 (S): now also U2.3 (SOURCE)
- net at Q19.1 (G), R24.1, R27.1: now also U6.2 (GATE)
- net at Q18.1 (G), R20.1, R21.1: now also U9.2 (GATE)
- net at Q17.3 (S), Q18.3 (S): now also U9.3 (SOURCE)
- net at C15.1, R30.1: now also U6.6 (GND)
- net at C15.2: now also U6.5 (INTVCC)
- net at C17.1, R33.1: now also U7.6 (GND)
- net at C17.2: now also U7.5 (INTVCC)
- net at C13.1, R28.1: now also U4.6 (GND)
- net at C13.2: now also U4.5 (INTVCC)
- net at Q13.1 (G), R19.1, R25.1: now also U4.2 (GATE)
- net at Q13.3 (S), Q14.3 (S): now also U4.3 (SOURCE)
- net at Q19.3 (S), Q20.3 (S): now also U6.3 (SOURCE)
- net 5V_REF_1 renamed 3.3V
- net 3.3V: now also C29.1, U12.13 (VD), U1.5 (OUT); no longer C18.1, C19.1, U8.2 (VA)
- net 5V_REF_2 renamed 5V_REGULATED
- net 5V_REGULATED: now also C18.1, C19.1, U8.2 (VA), PS2.6 (-VOUT), U1.1 (IN); no longer C29.1, U12.13 (VD)
- new net: C18.2, C19.2
- new net: C26.2, C27.2
- new net 24V_GND: J_ROCKET1.1 (Pin_1)
- new net 24V_REGULATED: J_ROCKET1.2 (Pin_2)
- new net 24_REGULATED: PS1.4 (+VOUT)
- new net ADC_2_CS: J19.1 (Pin_1), U12.1 (~{CS})
- new net ADC_2_DIN: J19.3 (Pin_3), U12.14 (DIN)
- new net ADC_2_DOUT: J19.4 (Pin_4), U12.15 (DOUT)
- new net ADC_2_SCLK: J19.2 (Pin_2), U12.16 (SCLK)
- new net GNDD: U12.12 (DGND), U8.12 (DGND)
Other:
- note added: "Buck Converters"
- note added: "Output connectors"
- moved on the sheet: C10, C12, C13, C14, C15, C16, C17, C18, C19, C3, C4, C5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

Commit message: updated resistor values
Parts:
- R14, R17, R21, R25, R26, R27, R32: value R -> 1K
- R36, R37, R38, R39, R4, R40, R41, R42: value R -> 2.7K
Changed lines of the file:
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@@
 		(fields_autoplaced yes)
 		(property "Reference" "R26"
-			(at 306.07 96.52 0)
+			(at 306.07 96.5199 0)
 			(effects
 				(font
@@
 			)
 		)
-		(property "Value" "R"
-			(at 306.07 99.06 0)
+		(property "Value" "1K"
+			(at 306.07 99.0599 0)
 			(effects
 				(font
@@
 		(fields_autoplaced yes)
 		(property "Reference" "R41"
-			(at 447.04 162.56 0)
+			(at 447.04 162.5599 0)
 			(effects
 				(font
@@
 			)
 		)
-		(property "Value" "R"
-			(at 447.04 165.1 0)
+		(property "Value" "2.7K"
+			(at 447.04 165.0999 0)
 			(effects
 				(font
@@
 		(fields_autoplaced yes)
 		(property "Reference" "R27"
-			(at 306.07 143.51 0)
+			(at 306.07 143.5099 0)
 			(effects
 				(font
@@
 			)
 		)
-		(property "Value" "R"
-			(at 306.07 146.05 0)
+		(property "Value" "1K"
+			(at 306.07 146.0499 0)
 			(effects
 				(font
@@
 		(fields_autoplaced yes)
 		(property "Reference" "R40"
-			(at 447.04 140.97 0)
+			(at 447.04 140.9699 0)
 			(effects
 				(font
@@
 			)
 		)
-		(property "Value" "R"
-			(at 447.04 143.51 0)
+		(property "Value" "2.7K"
+			(at 447.04 143.5099 0)
 			(effects
 				(font
@@
 		(fields_autoplaced yes)
 		(property "Reference" "R36"
-			(at 411.48 140.97 0)
+			(at 411.48 140.9699 0)
 			(effects
 				(font
@@
 			)
 		)
-		(property "Value" "R"
-			(at 411.48 143.51 0)
+		(property "Value" "2.7K"
+			(at 411.48 143.5099 0)
 			(effects
 				(font
@@
 		(fields_autoplaced yes)
 		(property "Reference" "R39"
-			(at 447.04 119.38 0)
+			(at 447.04 119.3799 0)
 			(effects
 				(font
@@
 			)
 		)
-		(property "Value" "R"
-			(at 447.04 121.92 0)
+		(property "Value" "2.7K"
+			(at 447.04 121.9199 0)
 			(effects
 				(font
@@
 		(fields_autoplaced yes)
 		(property "Reference" "R37"
-			(at 411.48 162.56 0)
+			(at 411.48 162.5599 0)
 			(effects
 				(font
@@
 			)
 		)
-		(property "Value" "R"
-			(at 411.48 165.1 0)
+		(property "Value" "2.7K"
+			(at 411.48 165.0999 0)
 			(effects
 				(font
@@
 		(fields_autoplaced yes)
 		(property "Reference" "R4"
-			(at 411.48 119.38 0)
+			(at 411.48 119.3799 0)
 			(effects
 				(font
@@
 			)
 		)
-		(property "Value" "R"
-			(at 411.48 121.92 0)
+		(property "Value" "2.7K"
+			(at 411.48 121.9199 0)
 			(effects
 				(font
@@
 		(fields_autoplaced yes)
 		(property "Reference" "R32"
-			(at 309.88 49.53 0)
+			(at 309.88 49.5299 0)
 			(effects
 				(font
@@
 			)
 		)
-		(property "Value" "R"
-			(at 309.88 52.07 0)
+		(property "Value" "1K"
+			(at 309.88 52.0699 0)
 			(effects
 				(font
@@
 		(fields_autoplaced yes)
 		(property "Reference" "R42"
-			(at 447.04 184.15 0)
+			(at 447.04 184.1499 0)
 			(effects
 				(font
@@
 			)
 		)
-		(property "Value" "R"
-			(at 447.04 186.69 0)
+		(property "Value" "2.7K"
+			(at 447.04 186.6899 0)
 			(effects
 				(font
@@
 		(fields_autoplaced yes)
 		(property "Reference" "R14"
-			(at 181.61 143.51 0)
+			(at 181.61 143.5099 0)
 			(effects
 				(font
@@
 			)
 		)
-		(property "Value" "R"
-			(at 181.61 146.05 0)
+		(property "Value" "1K"
+			(at 181.61 146.0499 0)
 			(effects
 				(font
@@
 		(fields_autoplaced yes)
 		(property "Reference" "R21"
-			(at 181.61 49.53 0)
+			(at 181.61 49.5299 0)
 			(effects
 				(font
@@
 			)
 		)
-		(property "Value" "R"
-			(at 181.61 52.07 0)
+		(property "Value" "1K"
+			(at 181.61 52.0699 0)
 			(effects
 				(font
@@
 		(fields_autoplaced yes)
 		(property "Reference" "R25"
-			(at 181.61 96.52 0)
+			(at 181.61 96.5199 0)
 			(effects
 				(font
@@
 			)
 		)
-		(property "Value" "R"
-			(at 181.61 99.06 0)
+		(property "Value" "1K"
+			(at 181.61 99.0599 0)
 			(effects
 				(font
@@
 		(fields_autoplaced yes)
 		(property "Reference" "R17"
-			(at 181.61 189.23 0)
+			(at 181.61 189.2299 0)
 			(effects
 				(font
@@
 			)
 		)
-		(property "Value" "R"
-			(at 181.61 191.77 0)
+		(property "Value" "1K"
+			(at 181.61 191.7699 0)
 			(effects
 				(font
@@
 		(fields_autoplaced yes)
 		(property "Reference" "R38"
-			(at 411.48 184.15 0)
+			(at 411.48 184.1499 0)
 			(effects
 				(font
@@
 			)
 		)
-		(property "Value" "R"
-			(at 411.48 186.69 0)
+		(property "Value" "2.7K"
+			(at 411.48 186.6899 0)
 			(effects
 				(font

Commit message: added resistor and capacitor footprints
Parts:
- removed C24, C25: 330 uF, symbol Device:C
- added C24, C25: UVZ2A331MHD1TO, UVZ2A331MHD:CAP_UEP_12P5X25_NCH, symbol 2025-11-07_01-42-20:UVZ2A331MHD1TO
- C1, C10, C11, C12, C13, C14, C15, C16, C17, C18, C19, C2, C20, C21, C22, C23, C26, C27, C3, C4, C5, C6, C7, C8, C9: footprint (none) -> Capacitor_SMD:C_0201_0603Metric_Pad0.64x0.40mm_HandSolder
- C28, C29: value C -> 1uF; footprint (none) -> Capacitor_SMD:C_0201_0603Metric_Pad0.64x0.40mm_HandSolder
- R1, R13, R14, R15, R16, R17, R18, R19, R2, R20, R21, R22, R23, R24, R25, R26, R27, R28, R29, R3, R30, R31, R32, R33, R34, R35, R36, R37, R38, R39, R4, R40, R41, R42: footprint (none) -> Resistor_SMD:R_0805_2012Metric_Pad1.20x1.40mm_HandSolder
Connections:
- net 24V_UNREGULATED: now also C24.1, C25.1
- net GND: now also C24.2, C25.2
Other:
- moved on the sheet: C29

Commit message: connectors update
Parts:
- removed J_JETSON1, J_PIX1, J_PIX2, J_SERVO1: Conn_01x02, symbol Connector_Generic:Conn_01x02
- removed TP1, TP2, TP3, TP4, TP5, TP6, TP7, TP8, TP9: TestPoint, TestPoint:TestPoint_Pad_1.5x1.5mm, symbol Connector:TestPoint
- added J_Motor1, J_Motor2: Conn_01x02, Connector_AMASS:AMASS_XT60PW-F_1x02_P7.20mm_Horizontal, symbol Connector_Generic:Conn_01x02
- J19, J20: footprint (none) -> Connector_Molex:Molex_Micro-Fit_3.0_43045-0400_2x02_P3.00mm_Horizontal
- J_ROCKET1: footprint (none) -> Connector_AMASS:AMASS_XT30UPB-F_1x02_P5.0mm_Vertical
Connections:
- net 24V_GND is gone; now on net GND: J_ROCKET1.1 (Pin_1)
- net 12V_UNREGULATED: now also J_Motor1.2 (Pin_2), J_Motor2.2 (Pin_2)
- net GND: now also J_Motor1.1 (Pin_1), J_Motor2.1 (Pin_1)
