File: Power Board/Power Board.kicad_pcb (KiCad board)
At the start: 2 copper layers, 150 parts, among them IC1 LTC4151IMS#PBF, J1 Conn_01x02, J10 Conn_01x02, J11 Conn_01x02, J12 Conn_01x02, J13 Conn_01x02, J14 Conn_01x02, J15 Conn_01x02, J16 Conn_01x02, J17 Conn_01x02, J2 Conn_01x02, J3 Conn_01x02, J4 Conn_01x02, J5 Conn_01x02, J6 Conn_01x02, J7 Conn_01x02, J8 Conn_01x02, Q1 Q_PMOS_GDS, Q10 Q_NMOS_GDS, Q11 Q_NMOS_GDS, Q12 Q_NMOS_GDS, Q13 Q_NMOS_GDS, Q14 Q_NMOS_GDS, Q15 Q_NMOS_GDS, Q16 Q_NMOS_GDS, Q17 Q_NMOS_GDS, Q18 Q_NMOS_GDS, Q19 Q_NMOS_GDS, Q2 Q_PMOS_GDS, Q20 Q_NMOS_GDS, Q21 Q_NMOS_GDS, Q22 Q_NMOS_GDS, Q3 Q_PMOS_GDS, Q4 Q_PMOS_GDS, Q5 Q_PMOS_GDS, Q6 Q_PMOS_GDS, Q7 Q_PMOS_GDS, Q8 Q_PMOS_GDS, Q9 Q_NMOS_GDS, U1 TLV70033_SOT23-5, U11 ACS770xCB-200U-PFF, U12 ADC128S052CIMT, U2 LTC4372CDD-PBF, U3 LTC4372CDD-PBF, U4 LTC4372CDD-PBF, U5 LTC4372CDD-PBF, U6 LTC4372CDD-PBF, U7 LTC4372CDD-PBF, U8 ADC128S052CIMT, U9 LTC4372CDD-PBF

Commit message: connectors update
Parts:
- removed TP1, TP2, TP3, TP4, TP5, TP6, TP7, TP8, TP9: TestPoint, TestPoint:TestPoint_Pad_1.5x1.5mm
- added J19: Conn_01x04, Connector_Molex:Molex_Micro-Fit_3.0_43045-0400_2x02_P3.00mm_Horizontal, F.Cu at (195.8, 113.3)
- added J20: Conn_01x04, Connector_Molex:Molex_Micro-Fit_3.0_43045-0400_2x02_P3.00mm_Horizontal, F.Cu at (208.0, 113.3)
- added J_Motor1: Conn_01x02, Connector_AMASS:AMASS_XT60PW-F_1x02_P7.20mm_Horizontal, F.Cu at (203.6, 100.3)
- added J_Motor2: Conn_01x02, Connector_AMASS:AMASS_XT60PW-F_1x02_P7.20mm_Horizontal, F.Cu at (221.1, 100.3)
- added J_ROCKET1: Conn_01x02, Connector_AMASS:AMASS_XT30UPB-F_1x02_P5.0mm_Vertical, F.Cu at (219.2, 107.0)
- moved C24 87.3 mm to (187.9, 148.0)
- moved C25 53.8 mm to (239.9, 149.0)
- moved IC1 32.4 mm to (194.6, 129.5)
- moved PS2 24.2 mm to (169.0, 158.3)
- moved R1 24.0 mm to (232.1, 76.3)
- moved R13 24.0 mm to (232.1, 88.1)
- moved R14 24.0 mm to (232.1, 91.0)
- moved R15 24.0 mm to (232.1, 94.0)
- moved R16 24.0 mm to (232.1, 97.0)
- moved R17 24.0 mm to (232.1, 99.9)
- moved R18 24.0 mm to (236.9, 76.3)
- moved R19 24.0 mm to (236.9, 79.2)
- moved R2 24.0 mm to (232.1, 79.2)
- moved R20 24.0 mm to (236.9, 82.2)
- moved R21 24.0 mm to (236.9, 85.2)
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
Commit message: updated schematic numbering, made rough PCB design for battery 1
Parts:
- removed J_Motor1, J_Motor2: Conn_01x02, Connector_AMASS:AMASS_XT60PW-F_1x02_P7.20mm_Horizontal
- removed R30, R33: 100, Resistor_SMD:R_0805_2012Metric_Pad1.20x1.40mm_HandSolder
- removed R31: 10, Resistor_SMD:R_0805_2012Metric_Pad1.20x1.40mm_HandSolder
- removed R32: 1K, Resistor_SMD:R_0805_2012Metric_Pad1.20x1.40mm_HandSolder
- removed R34: 20k, Resistor_SMD:R_0805_2012Metric_Pad1.20x1.40mm_HandSolder
- removed R35: 10k, Resistor_SMD:R_0805_2012Metric_Pad1.20x1.40mm_HandSolder
- removed R36, R37, R38, R39, R40, R41, R42: 2.7K, Resistor_SMD:R_0805_2012Metric_Pad1.20x1.40mm_HandSolder
- added C30: 22 nF, Capacitor_SMD:C_0201_0603Metric_Pad0.64x0.40mm_HandSolder, F.Cu at (276.4, 92.3)
- added C31: 22 nF, Capacitor_SMD:C_0201_0603Metric_Pad0.64x0.40mm_HandSolder, F.Cu at (276.4, 94.1)
- added C32: 0.1 uF, Capacitor_SMD:C_0201_0603Metric_Pad0.64x0.40mm_HandSolder, F.Cu at (276.4, 95.8)
- added C33: 0.1 uF, Capacitor_SMD:C_0201_0603Metric_Pad0.64x0.40mm_HandSolder, F.Cu at (276.4, 97.6)
- added C34: 1 uF, Capacitor_SMD:C_0201_0603Metric_Pad0.64x0.40mm_HandSolder, F.Cu at (276.4, 99.3)
- added C35: 0.1 uF, Capacitor_SMD:C_0201_0603Metric_Pad0.64x0.40mm_HandSolder, F.Cu at (276.4, 101.1)
- added C36: 1 uF, Capacitor_SMD:C_0201_0603Metric_Pad0.64x0.40mm_HandSolder, F.Cu at (279.2, 92.3)
- added C37: 0.1 uF, Capacitor_SMD:C_0201_0603Metric_Pad0.64x0.40mm_HandSolder, F.Cu at (279.2, 94.1)
- added C38: 1 uF, Capacitor_SMD:C_0201_0603Metric_Pad0.64x0.40mm_HandSolder, F.Cu at (279.2, 95.8)
- added C39: 0.1 uF, Capacitor_SMD:C_0201_0603Metric_Pad0.64x0.40mm_HandSolder, F.Cu at (279.2, 97.6)
- added C40: 1 uF, Capacitor_SMD:C_0201_0603Metric_Pad0.64x0.40mm_HandSolder, F.Cu at (279.2, 99.3)
- added C41: 0.1 uF, Capacitor_SMD:C_0201_0603Metric_Pad0.64x0.40mm_HandSolder, F.Cu at (279.2, 101.1)
- added C42: 1 uF, Capacitor_SMD:C_0201_0603Metric_Pad0.64x0.40mm_HandSolder, F.Cu at (282.0, 92.3)
- added C43: 0.1 uF, Capacitor_SMD:C_0201_0603Metric_Pad0.64x0.40mm_HandSolder, F.Cu at (282.0, 94.1)
- added C44: 1 uF, Capacitor_SMD:C_0201_0603Metric_Pad0.64x0.40mm_HandSolder, F.Cu at (282.0, 95.8)
- added C45: 0.1 uF, Capacitor_SMD:C_0201_0603Metric_Pad0.64x0.40mm_HandSolder, F.Cu at (282.0, 97.6)
- added C46: 1 uF, Capacitor_SMD:C_0201_0603Metric_Pad0.64x0.40mm_HandSolder, F.Cu at (282.0, 99.3)
- added C47: 0.1 uF, Capacitor_SMD:C_0201_0603Metric_Pad0.64x0.40mm_HandSolder, F.Cu at (282.0, 101.1)
- added C48: 1 uF, Capacitor_SMD:C_0201_0603Metric_Pad0.64x0.40mm_HandSolder, F.Cu at (284.8, 92.3)
- added C49: 1uF, Capacitor_SMD:C_0201_0603Metric_Pad0.64x0.40mm_HandSolder, F.Cu at (284.8, 94.1)
- added C50: 1uF, Capacitor_SMD:C_0201_0603Metric_Pad0.64x0.40mm_HandSolder, F.Cu at (284.8, 95.8)
- added C51: UVZ2A331MHD1TO, Capacitor_SMD:C_0201_0603Metric_Pad0.64x0.40mm_HandSolder, F.Cu at (284.8, 97.6)
- added C52: UVZ2A331MHD1TO, Capacitor_SMD:C_0201_0603Metric_Pad0.64x0.40mm_HandSolder, F.Cu at (284.8, 99.3)
- added RA1: 100, Resistor_SMD:R_0805_2012Metric_Pad1.20x1.40mm_HandSolder, F.Cu at (70.8, 132.5)
- added RA10: 100, Resistor_SMD:R_0805_2012Metric_Pad1.20x1.40mm_HandSolder, F.Cu at (75.5, 135.4)
- added RA11: 100, Resistor_SMD:R_0805_2012Metric_Pad1.20x1.40mm_HandSolder, F.Cu at (75.5, 138.4)
- added RA12: 100, Resistor_SMD:R_0805_2012Metric_Pad1.20x1.40mm_HandSolder, F.Cu at (75.5, 141.3)
- added RA13: 100, Resistor_SMD:R_0805_2012Metric_Pad1.20x1.40mm_HandSolder, F.Cu at (75.5, 144.3)
- added RA14: 100, Resistor_SMD:R_0805_2012Metric_Pad1.20x1.40mm_HandSolder, F.Cu at (75.5, 147.2)
- added RA2: 100, Resistor_SMD:R_0805_2012Metric_Pad1.20x1.40mm_HandSolder, F.Cu at (70.8, 135.4)
- added RA3: 100, Resistor_SMD:R_0805_2012Metric_Pad1.20x1.40mm_HandSolder, F.Cu at (70.8, 138.4)
- added RA4: 100, Resistor_SMD:R_0805_2012Metric_Pad1.20x1.40mm_HandSolder, F.Cu at (70.8, 141.3)
- added RA5: 100, Resistor_SMD:R_0805_2012Metric_Pad1.20x1.40mm_HandSolder, F.Cu at (70.8, 144.3)
- added RA6: 100, Resistor_SMD:R_0805_2012Metric_Pad1.20x1.40mm_HandSolder, F.Cu at (70.8, 147.2)
- added RA7: 100, Resistor_SMD:R_0805_2012Metric_Pad1.20x1.40mm_HandSolder, F.Cu at (70.8, 150.2)
- added RA8: 100, Resistor_SMD:R_0805_2012Metric_Pad1.20x1.40mm_HandSolder, F.Cu at (70.8, 153.2)
- added RA9: 100, Resistor_SMD:R_0805_2012Metric_Pad1.20x1.40mm_HandSolder, F.Cu at (75.5, 132.5)
- added RI1: 0.04, Resistor_SMD:R_0805_2012Metric_Pad1.20x1.40mm_HandSolder, F.Cu at (75.5, 150.2)
- added RT1: 2.7K, Resistor_SMD:R_0805_2012Metric_Pad1.20x1.40mm_HandSolder, F.Cu at (75.5, 153.2)
- added RT2: 2.7K, Resistor_SMD:R_0805_2012Metric_Pad1.20x1.40mm_HandSolder, F.Cu at (80.3, 132.5)
- added RT3: 2.7K, Resistor_SMD:R_0805_2012Metric_Pad1.20x1.40mm_HandSolder, F.Cu at (80.3, 135.4)
- added RT4: 2.7K, Resistor_SMD:R_0805_2012Metric_Pad1.20x1.40mm_HandSolder, F.Cu at (80.3, 138.4)
- added RT5: 2.7K, Resistor_SMD:R_0805_2012Metric_Pad1.20x1.40mm_HandSolder, F.Cu at (80.3, 141.3)
- added RT6: 2.7K, Resistor_SMD:R_0805_2012Metric_Pad1.20x1.40mm_HandSolder, F.Cu at (80.3, 144.3)
- added RT7: 2.7K, Resistor_SMD:R_0805_2012Metric_Pad1.20x1.40mm_HandSolder, F.Cu at (80.3, 147.2)
- added RT8: 2.7K, Resistor_SMD:R_0805_2012Metric_Pad1.20x1.40mm_HandSolder, F.Cu at (80.3, 150.2)
- added U10: ACS770xCB-050U-PFF, Sensor_Current:Allegro_CB_PFF, F.Cu at (264.6, 90.0)
- added U13: ACS770xCB-050U-PFF, Sensor_Current:Allegro_CB_PFF, F.Cu at (285.2, 90.0)
- added U14: ACS770xCB-050U-PFF, Sensor_Current:Allegro_CB_PFF, F.Cu at (305.9, 90.0)
- added U15: ADC128S052CIMT, ADC128S052CIMT_NOPB:SOP65P640X120-16N, F.Cu at (270.5, 94.8)
- added U16: ADC128S052CIMT, ADC128S052CIMT_NOPB:SOP65P640X120-16N, F.Cu at (270.5, 101.3)
- added U17: TLV70033_SOT23-5, Package_TO_SOT_SMD:SOT-23-5, F.Cu at (277.6, 104.4)
- C1: value 22 nF -> 10nF
- C10: value 10 uF -> 100 nF
- C13: value 100 nF -> 10nF
- C15, C17: value 100 nF -> 22 nF
- C16: value 10nF -> 22 nF
- C18, C20, C21, C26: value 0.1 uF -> 22 nF
- C19, C27: value 1 uF -> 22 nF
- C2: value 22 nF -> 100 nF
- C23: value 1 uF -> 0.1 uF
- C24: value UVZ2A331MHD1TO -> 1 uF; footprint UVZ2A331MHD:CAP_UEP_12P5X25_NCH -> Capacitor_SMD:C_0201_0603Metric_Pad0.64x0.40mm_HandSolder
- C25: value UVZ2A331MHD1TO -> 22 nF; footprint UVZ2A331MHD:CAP_UEP_12P5X25_NCH -> Capacitor_SMD:C_0201_0603Metric_Pad0.64x0.40mm_HandSolder
- C28, C29: value 1uF -> 22 nF
- C8: value 10nF -> 100 nF
- R1: value 0.04 -> 100k
- R10: value 100k -> 1K
- R11: value 100k -> 100
- R12, R9: value 100k -> 10
- R13, R16, R19: value 10 -> 1K
- R14, R17, R26: value 1K -> 100
- R15, R18: value 100 -> 10
- R2, R3: value 100 -> 100k
- R20, R23: value 10 -> 100
- R21, R27: value 1K -> 10
- R22, R28: value 100 -> 1K
- R4: value 2.7K -> 100k
- U1: value TLV70033_SOT23-5 -> LTC4372CDD-PBF; footprint Package_TO_SOT_SMD:SOT-23-5 -> footprints:05-08-1698_ADI
- U11: value ACS770xCB-200U-PFF -> ACS770xCB-050U-PFF
- U12, U8: value ADC128S052CIMT -> ACS770xCB-050U-PFF; footprint ADC128S052CIMT_NOPB:SOP65P640X120-16N -> Sensor_Current:Allegro_CB_PFF
- U9: value LTC4372CDD-PBF -> ACS770xCB-050U-PFF; footprint footprints:05-08-1698_ADI -> Sensor_Current:Allegro_CB_PFF
- moved R20 143.7 mm to (93.2, 82.6)
- moved C2 132.2 mm to (113.4, 43.8), turned to 90 degrees
- moved R1 130.5 mm to (105.6, 44.3), turned to 180 degrees
- moved C1 126.6 mm to (124.5, 34.0), turned to -90 degrees
- moved Q10 120.4 mm to (113.3, 36.7), turned to 90 degrees
- moved R5 111.3 mm to (102.8, 152.8), turned to 180 degrees
- moved Q3 96.8 mm to (64.3, 140.8)
- moved Q4 96.4 mm to (64.3, 147.4)
- moved Q5 96.3 mm to (64.3, 153.9)
- moved Q6 95.9 mm to (64.3, 160.5)
- moved Q2 93.2 mm to (64.3, 134.3)
- moved Q7 90.6 mm to (64.3, 167.1)
- moved C10 86.1 mm to (156.0, 69.2)
- moved J5 79.6 mm to (124.9, 108.5), turned to 0 degrees
- moved U9 73.0 mm to (143.8, 105.0)
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Connections:
- C1 pad 1: Net-(U8-IN1) -> Net-(C1-Pad1)
- C10 pad 1: /12V_PSO -> Net-(C10-Pad1)
- C10 pad 2: GND -> Net-(U5-INTVCC)
- C12 pad 2: Net-(U9-INTVCC) -> Net-(U6-INTVCC)
- C13 pad 2: Net-(U4-INTVCC) -> GND
- C14 pad 2: Net-(U5-INTVCC) -> Net-(U7-INTVCC)
- C15 pad 1: Net-(C15-Pad1) -> Net-(U15-IN0)
- C15 pad 2: Net-(U6-INTVCC) -> GND
- C17 pad 1: Net-(C17-Pad1) -> Net-(U15-IN2)
- C17 pad 2: Net-(U7-INTVCC) -> GND
- C18 pad 1: /5V_REGULATED -> Net-(U15-IN3)
- C18 pad 2: Net-(C18-Pad2) -> GND
- C19 pad 1: /5V_REGULATED -> Net-(U15-IN4)
- C19 pad 2: Net-(C18-Pad2) -> GND
- C2 pad 1: Net-(U8-IN0) -> Net-(C2-Pad1)
- C2 pad 2: GND -> Net-(U1-INTVCC)
- C20 pad 1: /3.3V -> Net-(U15-IN5)
- C21 pad 1: /3.3V -> Net-(U15-IN6)
- C22 pad 1: +5V -> /3.3V
- C23 pad 1: +5V -> /5V_REGULATED
- C23 pad 2: GND -> Net-(C23-Pad2)
- C24 pad 1: /24V_UNREGULATED -> /5V_REGULATED
- C24 pad 2: GND -> Net-(C23-Pad2)
- C25 pad 1: /24V_UNREGULATED -> Net-(U16-IN0)
- C26 pad 1: /5V_REGULATED -> Net-(U16-IN1)
- C26 pad 2: Net-(C26-Pad2) -> GND
- C27 pad 1: /5V_REGULATED -> Net-(U16-IN2)
- C27 pad 2: Net-(C26-Pad2) -> GND
- C28 pad 1: /5V_REGULATED -> Net-(U16-IN3)
- C29 pad 1: /3.3V -> Net-(U16-IN4)
- C8 pad 2: GND -> Net-(U4-INTVCC)
- Q10 pad 2: /BATT_IN_12_2 -> /BATT_IN_12_1
- Q11 pad 2: /12V_PRESENSE -> /BATT_2_PRESENSE
- Q12 pad 2: /BATT_IN_12_3 -> /BATT_IN_12_4
- Q13 pad 2: /12V_PRESENSE -> /BATT_3_PRESENSE
- Q14 pad 2: /BATT_IN_12_4 -> /BATT_IN_12_2
- Q15 pad 2: /12V_PRESENSE -> /BATT_4_PRESENSE
- Q16 pad 2: /BATT_IN_12_5 -> /BATT_IN_12_3
- Q17 pad 2: /BATT_IN_12_1 -> /BATT_5_PRESENSE
- Q18 pad 2: /12V_PRESENSE -> /BATT_IN_12_7
- Q19 pad 2: /12V_PRESENSE -> /BATT_6_PRESENSE
- Q20 pad 2: /BATT_IN_12_6 -> /BATT_IN_12_5
- Q21 pad 2: /12V_PRESENSE -> /BATT_7_PRESENSE
- Q22 pad 2: /BATT_IN_12_7 -> /BATT_IN_12_6
- Q9 pad 2: /12V_PRESENSE -> /BATT_1_PRESENSE
- R1 pad 1: /24V_PRESENSE -> Net-(D1-A)
- R1 pad 2: /24V_UNREGULATED -> GND
- R10 pad 1: Net-(D6-A) -> Net-(Q9-G)
- R10 pad 2: GND -> Net-(C1-Pad1)
- R11 pad 1: Net-(D7-A) -> Net-(C2-Pad1)
- R12 pad 1: Net-(D8-A) -> Net-(Q11-G)
- R12 pad 2: GND -> Net-(Q12-G)
- R13 pad 1: Net-(Q9-G) -> Net-(Q11-G)
- R13 pad 2: Net-(Q10-G) -> Net-(C3-Pad1)
- R14 pad 1: Net-(Q9-G) -> Net-(C4-Pad1)
- R14 pad 2: Net-(C3-Pad1) -> GND
- R15 pad 1: Net-(C4-Pad1) -> Net-(Q13-G)
- R15 pad 2: GND -> Net-(Q14-G)
- R16 pad 1: Net-(Q11-G) -> Net-(Q13-G)
- R16 pad 2: Net-(Q12-G) -> Net-(C5-Pad1)
- R17 pad 1: Net-(Q11-G) -> Net-(C6-Pad1)
- R17 pad 2: Net-(C5-Pad1) -> GND
- R18 pad 1: Net-(C6-Pad1) -> Net-(Q15-G)
- R18 pad 2: GND -> Net-(Q16-G)
- R19 pad 1: Net-(Q13-G) -> Net-(Q15-G)
- R19 pad 2: Net-(Q14-G) -> Net-(C7-Pad1)
- R2 pad 1: Net-(R2-Pad1) -> Net-(D2-A)
- R2 pad 2: Net-(U8-IN1) -> GND
- R20 pad 1: Net-(Q18-G) -> Net-(C8-Pad1)
- R20 pad 2: Net-(Q17-G) -> GND
- R21 pad 1: Net-(Q18-G) -> Net-(Q17-G)
- R21 pad 2: Net-(C11-Pad1) -> Net-(Q18-G)
- R22 pad 1: Net-(C12-Pad1) -> Net-(Q17-G)
- R22 pad 2: GND -> Net-(C9-Pad1)
- R23 pad 1: Net-(Q15-G) -> Net-(C10-Pad1)
- R23 pad 2: Net-(Q16-G) -> GND
- R25 pad 1: Net-(Q13-G) -> Net-(Q19-G)
- R25 pad 2: Net-(C7-Pad1) -> Net-(C11-Pad1)
- R26 pad 1: Net-(Q15-G) -> Net-(C12-Pad1)
- R26 pad 2: Net-(C8-Pad1) -> GND
- R27 pad 1: Net-(Q19-G) -> Net-(Q21-G)
- R27 pad 2: Net-(C9-Pad1) -> Net-(Q22-G)
- R28 pad 1: Net-(C13-Pad1) -> Net-(Q21-G)
- R28 pad 2: GND -> Net-(C13-Pad1)
- R3 pad 1: /12V_AMP_SENSE -> Net-(D3-A)
- R3 pad 2: Net-(U8-IN0) -> GND
- R4 pad 1: /THERM_1 -> Net-(D4-A)
- R5 pad 1: Net-(D1-A) -> Net-(D5-A)
- R6 pad 1: Net-(D2-A) -> Net-(D6-A)
- R7 pad 1: Net-(D3-A) -> Net-(D7-A)
- R8 pad 1: Net-(D4-A) -> Net-(D8-A)
- R9 pad 1: Net-(D5-A) -> Net-(Q9-G)
- R9 pad 2: GND -> Net-(Q10-G)
- U1 pad 1: /5V_REGULATED -> /BATT_1_PRESENSE
- U1 pad 2: GND -> Net-(Q9-G)
- U1 pad 3: unconnected-(U1-EN-Pad3) -> Net-(Q10-S)
- U1 pad 4: unconnected-(U1-NC-Pad4) -> /BATT_IN_12_1
- U1 pad 5: /3.3V -> Net-(U1-INTVCC)
- U11 pad 1: +5V -> /5V_REGULATED
- U11 pad 3: /12V_AMP_SENSE -> /BATT_4_SENSE
- U11 pad 4: /12V_PRESENSE -> /BATT_4_PRESENSE
- U11 pad 5: /12V_UNREGULATED -> /BATT_4
- U12 pad 1: /ADC_2_CS -> /5V_REGULATED
- U12 pad 2: /5V_REGULATED -> GND
- U12 pad 3: GND -> /BATT_5_SENSE
- U12 pad 4: /THERM_1 -> /BATT_5_PRESENSE
- U12 pad 5: /THERM_2 -> /BATT_5
- U2 pad 1: /12V_PRESENSE -> /BATT_2_PRESENSE
- U2 pad 2: Net-(Q9-G) -> Net-(Q11-G)
- U2 pad 3: Net-(Q10-S) -> Net-(Q11-S)
- U2 pad 4: /BATT_IN_12_2 -> /BATT_IN_12_4
- U3 pad 1: /12V_PRESENSE -> /BATT_3_PRESENSE
- U3 pad 2: Net-(Q11-G) -> Net-(Q13-G)
- U3 pad 3: Net-(Q11-S) -> Net-(Q13-S)
- U3 pad 4: /BATT_IN_12_3 -> /BATT_IN_12_2
- U4 pad 1: /12V_PRESENSE -> /BATT_4_PRESENSE
- U4 pad 2: Net-(Q13-G) -> Net-(Q15-G)
- U4 pad 3: Net-(Q13-S) -> Net-(Q15-S)
- U4 pad 4: /BATT_IN_12_4 -> /BATT_IN_12_3
- U4 pad 6: Net-(C13-Pad1) -> Net-(C8-Pad1)
- U5 pad 1: unconnected-(U5-OUT-Pad1) -> /BATT_5_PRESENSE
- U5 pad 2: unconnected-(U5-GATE-Pad2) -> Net-(Q17-G)
- U5 pad 3: unconnected-(U5-SOURCE-Pad3) -> Net-(Q17-S)
- U5 pad 4: /BATT_IN_12_5 -> /BATT_IN_12_7
- U5 pad 6: Net-(C14-Pad1) -> Net-(C10-Pad1)
- U6 pad 1: /12V_PRESENSE -> unconnected-(U6-OUT-Pad1)
- U6 pad 2: Net-(Q19-G) -> unconnected-(U6-GATE-Pad2)
- U6 pad 3: Net-(Q19-S) -> unconnected-(U6-SOURCE-Pad3)
- U6 pad 4: /BATT_IN_12_6 -> /BATT_IN_12_5
- U6 pad 6: Net-(C15-Pad1) -> Net-(C12-Pad1)
- U7 pad 1: /12V_PRESENSE -> /BATT_7_PRESENSE
- U7 pad 4: /BATT_IN_12_7 -> /BATT_IN_12_6
- U7 pad 6: Net-(C17-Pad1) -> Net-(C14-Pad1)
- U8 pad 1: /ADC_1_CS -> /5V_REGULATED
- U8 pad 2: /5V_REGULATED -> GND
- U8 pad 3: GND -> /BATT_1_SENSE
- U8 pad 4: Net-(U8-IN0) -> /BATT_1_PRESENSE
- U8 pad 5: Net-(U8-IN1) -> /BATT_1
- U9 pad 1: /12V_PRESENSE -> /5V_REGULATED
- U9 pad 2: Net-(Q18-G) -> GND
- U9 pad 3: Net-(Q17-S) -> /BATT_2_SENSE
- U9 pad 4: /BATT_IN_12_1 -> /BATT_2_PRESENSE
- U9 pad 5: Net-(U9-INTVCC) -> /BATT_2
Routing:
- net /BATT_1: track 0.00 -> 63.7 mm
- net Net-(J6-Pin_2): track 24.9 -> 0.00 mm
- net Net-(J8-Pin_2): track 24.4 -> 0.00 mm
- net Net-(J2-Pin_2): track 24.3 -> 0.00 mm
- net Net-(J7-Pin_2): track 24.2 -> 0.00 mm
- net Net-(J3-Pin_2): track 23.8 -> 0.00 mm
- net Net-(J5-Pin_2): track 23.6 -> 0.00 mm
- net /BATT_1_PRESENSE: track 0.00 -> 23.3 mm, vias 0 -> 1
- net Net-(J4-Pin_2): track 23.1 -> 0.00 mm
- net /BATT_IN_12_1: track 0.00 -> 14.5 mm, vias 0 -> 2
- net Net-(Q10-G): track 0.00 -> 13.4 mm
- net Net-(Q1-D): track 2.50 -> 15.9 mm, vias 0 -> 1
- net Net-(D1-A): track 0.00 -> 12.3 mm
- net Net-(Q10-S): track 0.00 -> 10.7 mm, vias 0 -> 1
- net Net-(C2-Pad1): track 0.00 -> 7.11 mm
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
Commit message: adc design on power board
Parts:
- removed the D2 at (158.9, 93.7)
- removed the F2 at (38.8, 98.7)
- removed the J2 at (72.2, 108.5)
- removed the Q11 at (233.4, 36.1)
- removed the Q12 at (233.4, 42.9)
- removed the Q2 at (64.3, 134.3)
- removed the R12 at (178.5, 55.2)
- removed the RT2 at (80.3, 132.5)
- removed the U2 at (257.1, 21.8)
- removed the U9 at (143.8, 105.0)
- added C1: 10nF, Capacitor_SMD:C_0201_0603Metric_Pad0.64x0.40mm_HandSolder, F.Cu at (124.5, 56.3)
- added C4: 100 nF, Capacitor_SMD:C_0201_0603Metric_Pad0.64x0.40mm_HandSolder, F.Cu at (113.4, 66.1)
- added D2: D_Zener, Diode_SMD:D_SOD-123, F.Cu at (-57.4, 310.7)
- added D2: D_Zener, Diode_SMD:D_SOD-123, F.Cu at (110.3, 66.3)
- added F2: Fuse, 0498060:Fuse_0498060M, F.Cu at (82.5, 61.2)
- added F2: Fuse, 0498060:Fuse_0498060M, F.Cu at (-128.5, 250.0)
- added J11: Conn_01x02, Connector_Molex:Molex_KK-254_AE-6410-02A_1x02_P2.54mm_Vertical, F.Cu at (123.6, 68.9)
- added J2: Conn_01x02, Connector_AMASS:AMASS_XT60PW-F_1x02_P7.20mm_Horizontal, F.Cu at (45.5, 64.6)
- added J2: Conn_01x02, Connector_AMASS:AMASS_XT60PW-F_1x02_P7.20mm_Horizontal, F.Cu at (-95.1, 259.8)
- added Q11: Q_NMOS_GDS, Package_TO_SOT_SMD:TDSON-8-1, F.Cu at (-94.8, 312.4)
- added Q11: Q_NMOS_GDS, Package_TO_SOT_SMD:TDSON-8-1, F.Cu at (122.2, 60.5)
- added Q12: Q_NMOS_GDS, Package_TO_SOT_SMD:TDSON-8-1, F.Cu at (113.3, 58.9)
- added Q12: Q_NMOS_GDS, Package_TO_SOT_SMD:TDSON-8-1, F.Cu at (-94.8, 319.1)
- added Q2: Q_PMOS_GDS, Package_SO:PowerPAK_SO-8_Single, F.Cu at (-103.0, 312.3)
- added Q2: Q_PMOS_GDS, Package_SO:PowerPAK_SO-8_Single, F.Cu at (106.9, 58.9)
- added R12: 10, Resistor_SMD:R_0805_2012Metric_Pad1.20x1.40mm_HandSolder, F.Cu at (-52.2, 322.3)
- added R12: 10, Resistor_SMD:R_0805_2012Metric_Pad1.20x1.40mm_HandSolder, F.Cu at (118.2, 56.3)
- added R13: 1K, Resistor_SMD:R_0805_2012Metric_Pad1.20x1.40mm_HandSolder, F.Cu at (122.1, 56.3)
- added R14: 100, Resistor_SMD:R_0805_2012Metric_Pad1.20x1.40mm_HandSolder, F.Cu at (119.0, 65.5)
- added R2: 100k, Resistor_SMD:R_0805_2012Metric_Pad1.20x1.40mm_HandSolder, F.Cu at (105.6, 66.5)
- added RT2: 2.7K, Resistor_SMD:R_0805_2012Metric_Pad1.20x1.40mm_HandSolder, F.Cu at (-42.7, 310.5)
- added RT2: 2.7K, Resistor_SMD:R_0805_2012Metric_Pad1.20x1.40mm_HandSolder, F.Cu at (117.7, 69.5)
- added U2: LTC4372CDD-PBF, footprints:05-08-1698_ADI, F.Cu at (-63.0, 311.4)
- added U2: LTC4372CDD-PBF, footprints:05-08-1698_ADI, F.Cu at (115.8, 65.2)
- added U9: ACS770xCB-050U-PFF, Sensor_Current:Allegro_CB_PFF, F.Cu at (152.3, 62.8)
- added U9: ACS770xCB-050U-PFF, Sensor_Current:Allegro_CB_PFF, F.Cu at (-99.0, 307.5)
- C51, C52: value UVZ2A331MHD1TO -> EEV-TG2A331M; footprint Capacitor_SMD:C_0201_0603Metric_Pad0.64x0.40mm_HandSolder -> EEV_TG2A331M:CAP_SMD_19X19_PAN
- moved Q19 446.8 mm to (-78.4, 325.8)
- moved Q14 437.8 mm to (-86.6, 312.4)
- moved Q16 437.8 mm to (-86.6, 325.8)
- moved Q15 437.8 mm to (-86.6, 319.1)
- moved U3 431.7 mm to (-63.0, 316.2)
- moved U4 431.7 mm to (-63.0, 320.9)
- moved U5 431.7 mm to (-63.0, 325.7)
- moved U6 431.7 mm to (-63.0, 330.4)
- moved U7 431.7 mm to (-63.0, 335.2)
- moved Q13 429.0 mm to (-94.8, 325.8)
- moved Q20 427.2 mm to (-70.2, 312.4)
- moved Q21 427.2 mm to (-70.2, 319.1)
- moved Q22 427.2 mm to (-70.2, 325.8)
- moved U11 372.5 mm to (-78.4, 307.5)
- moved R6 359.7 mm to (-52.2, 313.4)
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Connections:
- C23 pad 2: Net-(C23-Pad2) -> GND
- C24 pad 2: Net-(C23-Pad2) -> GND
- C33 pad 2: Net-(C33-Pad2) -> GND
- C34 pad 2: Net-(C33-Pad2) -> GND
- C51 pad 1: /24V_UNREGULATED -> GND
- C51 pad 2: GND -> /24V_UNREGULATED
- IC1 pad 1: /24V_PRESENSE -> /24V_PSO
- IC1 pad 2: /24V_PRESENSE -> /24V_PSO
- IC1 pad 3: /24V_PRESENSE -> /24V_PSO
- PS1 pad 4: /24_REGULATED -> /24V_REGULATED
- RI1 pad 1: /24V_PRESENSE -> /24V_PSO
Routing:
- net /BATT_1: track 63.7 -> 19.1 mm
- net /24V_UNREGULATED: track 0.00 -> 34.5 mm
- net /ADC_1_CS: track 0.00 -> 31.3 mm
- net Net-(J2-Pin_2): track 0.00 -> 24.1 mm
- net /BATT_1_PRESENSE: track 23.3 -> 46.7 mm, vias 1 -> 2
- net /ADC_1_DIN: track 0.00 -> 23.2 mm
- net /ADC_1_DOUT: track 0.00 -> 21.9 mm
- net /3.3V: track 0.00 -> 21.7 mm
- net /BATT_2: track 0.00 -> 19.1 mm
- net /ADC_1_SCLK: track 0.00 -> 18.2 mm
- net /5V_REGULATED: track 0.00 -> 16.5 mm
- net Net-(Q2-D): track 0.00 -> 15.9 mm, vias 0 -> 1
- net /BATT_IN_12_1: track 14.5 -> 29.0 mm, vias 2 -> 4
- net Net-(Q12-G): track 0.00 -> 13.4 mm
- net Net-(D2-A): track 0.00 -> 12.3 mm
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
Commit message: laid out most components, reworked battery 1 pours, made connections for ADCs; buck converter layout and routing in progress
Parts:
- removed the C1 at (124.5, 56.3)
- removed the C4 at (113.4, 66.1)
- removed the D2 at (110.3, 66.3)
- removed the F2 at (82.5, 61.2)
- removed the J11 at (123.6, 68.9)
- removed the J2 at (45.5, 64.6)
- removed the Q11 at (122.2, 60.5)
- removed the Q12 at (113.3, 58.9)
- removed the Q2 at (106.9, 58.9)
- removed the R12 at (118.2, 56.3)
- removed the R13 at (122.1, 56.3)
- removed the R14 at (119.0, 65.5)
- removed the R2 at (105.6, 66.5)
- removed the RT2 at (-42.7, 310.5)
- removed the RT2 at (117.7, 69.5)
- removed the U2 at (115.8, 65.2)
- removed the U9 at (152.3, 62.8)
- added RT2: 2.7K, Resistor_SMD:R_0805_2012Metric_Pad1.20x1.40mm_HandSolder, F.Cu at (90.0, 73.8)
- Q10, Q11, Q12, Q13, Q14, Q15, Q16, Q17, Q18, Q19, Q20, Q21, Q22, Q9: footprint Package_TO_SOT_SMD:TDSON-8-1 -> Package_SO:PowerPAK_SO-8_Single
- moved U9 350.8 mm to (155.5, 66.1), turned to 90 degrees
- moved RA14 328.3 mm to (272.5, 251.3), turned to 180 degrees
- moved Q2 326.8 mm to (106.4, 61.5), turned to 90 degrees
- moved Q11 325.4 mm to (123.9, 71.5), turned to -90 degrees
- moved Q12 325.0 mm to (115.7, 71.5), turned to -90 degrees
- moved RA13 324.1 mm to (269.3, 253.5)
- moved RA8 321.2 mm to (258.7, 247.5)
- moved RA12 318.8 mm to (264.5, 253.5)
- moved Q13 317.1 mm to (124.2, 96.5), turned to -90 degrees
- moved Q3 312.8 mm to (106.4, 86.5), turned to 90 degrees
- moved RA11 312.2 mm to (258.7, 255.0)
- moved RA9 312.1 mm to (258.7, 249.5)
- moved RA10 312.0 mm to (258.7, 253.0)
- moved U2 310.7 mm to (120.8, 60.9)
- moved R12 305.8 mm to (112.4, 64.6), turned to 90 degrees
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Connections:
- C22 pad 2: GND -> GNDD
- C32 pad 2: GND -> GNDD
- J19 pad 2: /ADC_2_SCLK -> /ADC_2_DOUT
- J19 pad 3: /ADC_2_DIN -> /ADC_2_SCLK
- J19 pad 4: /ADC_2_DOUT -> /ADC_2_DIN
- J20 pad 2: /ADC_1_SCLK -> /ADC_1_DOUT
- J20 pad 3: /ADC_1_DIN -> /ADC_1_SCLK
- J20 pad 4: /ADC_1_DOUT -> /ADC_1_DIN
- U1 pad 9: unconnected-(U1-GND-Pad9) -> GND
- U2 pad 9: unconnected-(U2-GND-Pad9) -> GND
- U3 pad 9: unconnected-(U3-GND-Pad9) -> GND
- U4 pad 9: unconnected-(U4-GND-Pad9) -> GND
- U5 pad 9: unconnected-(U5-GND-Pad9) -> GND
- U6 pad 9: unconnected-(U6-GND-Pad9) -> GND
- U7 pad 9: unconnected-(U7-GND-Pad9) -> GND
Routing:
- net /5V_REGULATED: track 16.5 -> 88.5 mm, vias 0 -> 2
- net /24V_UNREGULATED: track 34.5 -> 101.0 mm
- net GND: track 0.00 -> 53.9 mm, vias 0 -> 30
- net /BATT_1_PRESENSE: track 46.7 -> 1.82 mm, vias 2 -> 21
- net /BATT_IN_12_1: track 29.0 -> 1.59 mm, vias 4 -> 24
- net Net-(J2-Pin_2): track 24.1 -> 0.00 mm
- net Net-(J1-Pin_2): track 24.1 -> 0.50 mm
- net /ADC_2_CS: track 0.00 -> 21.6 mm, vias 0 -> 1
- net /BATT_2: track 19.1 -> 0.00 mm
- net /BATT_1: track 19.1 -> 0.00 mm
- net /3.3V: track 21.7 -> 3.12 mm, vias 0 -> 2
- net Net-(Q2-D): track 15.9 -> 0.00 mm, vias 1 -> 0
- net Net-(Q9-G): track 6.18 -> 21.9 mm, vias 0 -> 3
- net /ADC_2_DOUT: track 0.00 -> 15.5 mm, vias 0 -> 1
- net Net-(Q12-G): track 13.4 -> 0.00 mm
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- added copper zone on F.Cu, net /24V_REGULATED
- added copper zone on F.Cu, net /5V_REGULATED
- added copper zone on In2.Cu, net /5V_REGULATED
- added copper zone on F.Cu, net /BATT_1
- added copper zone on B.Cu, net /BATT_1_PRESENSE
- added copper zone on F.Cu, net /BATT_1_PRESENSE
- added copper zone on B.Cu, net /BATT_IN_12_1
- added copper zone on F.Cu, net /BATT_IN_12_1
- added copper zone on F.Cu, net GND
- added copper zone on In1.Cu, net GND
- added copper zone on In1.Cu, net GNDD
- added copper zone on B.Cu, net Net-(J1-Pin_2)
- added copper zone on F.Cu, net Net-(J1-Pin_2)
- added copper zone on F.Cu, net Net-(J2-Pin_2)
- added copper zone on B.Cu, net Net-(Q1-D)
- added copper zone on F.Cu, net Net-(Q1-D)
- added copper zone on F.Cu, net Net-(Q10-S)
Other:
- copper layers 2 -> 4

Commit message: changed ADC connectors, added series resistors
Parts:
- removed J19: Conn_01x04, Connector_Molex:Molex_Micro-Fit_3.0_43045-0400_2x02_P3.00mm_Horizontal
- added J18: Conn_02x03_Top_Bottom, Connector_Molex:Molex_Nano-Fit_105310-xx06_2x03_P2.50mm_Vertical, F.Cu at (122.7, 213.6)
- added J9: Conn_02x03_Top_Bottom, Connector_Molex:Molex_Nano-Fit_105314-xx06_2x03_P2.50mm_Horizontal, F.Cu at (284.6, 227.8)
- added R30: 33, Resistor_SMD:R_0805_2012Metric_Pad1.20x1.40mm_HandSolder, F.Cu at (271.2, 223.7)
- added R31: 33, Resistor_SMD:R_0805_2012Metric_Pad1.20x1.40mm_HandSolder, F.Cu at (277.6, 228.0)
- added R32: 33, Resistor_SMD:R_0805_2012Metric_Pad1.20x1.40mm_HandSolder, F.Cu at (279.6, 233.1)
- added R33: 33, Resistor_SMD:R_0805_2012Metric_Pad1.20x1.40mm_HandSolder, F.Cu at (277.6, 225.2)
- added R34: 33, Resistor_SMD:R_0805_2012Metric_Pad1.20x1.40mm_HandSolder, F.Cu at (277.6, 243.6)
- added R35: 33, Resistor_SMD:R_0805_2012Metric_Pad1.20x1.40mm_HandSolder, F.Cu at (279.6, 251.5)
- added R36: 33, Resistor_SMD:R_0805_2012Metric_Pad1.20x1.40mm_HandSolder, F.Cu at (277.6, 246.4)
- added R37: 33, Resistor_SMD:R_0805_2012Metric_Pad1.20x1.40mm_HandSolder, F.Cu at (271.2, 242.1)
- J20: value Conn_01x04 -> Conn_02x03_Top_Bottom; footprint Connector_Molex:Molex_Micro-Fit_3.0_43045-0400_2x02_P3.00mm_Horizontal -> Connector_Molex:Molex_Nano-Fit_105314-xx06_2x03_P2.50mm_Horizontal
- moved D10 38.2 mm to (205.0, 237.9)
- moved D9 38.2 mm to (215.8, 237.9)
- moved C52 31.3 mm to (169.7, 218.6)
- moved PS2 31.3 mm to (141.1, 208.4)
- moved C51 30.8 mm to (170.0, 252.2)
- moved PS1 30.8 mm to (143.1, 249.5)
- moved J20 17.6 mm to (284.4, 246.2), turned to 0 degrees
- moved IC1 12.1 mm to (112.7, 234.9)
- moved C49 5.60 mm to (234.5, 240.1)
- moved U17 5.60 mm to (239.2, 240.8)
- moved C50 5.60 mm to (242.9, 240.2)
- moved RI1 5.01 mm to (112.7, 231.4)
- moved C25 1.15 mm to (260.1, 244.9)
- moved C26 1.15 mm to (260.1, 250.3)
- moved C27 1.15 mm to (258.3, 250.3)
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Connections:
- J20 pad 1: /ADC_1_CS -> Net-(J20-Pin_1)
- J20 pad 2: /ADC_1_DOUT -> GNDD
- J20 pad 3: /ADC_1_SCLK -> Net-(J20-Pin_3)
- J20 pad 4: /ADC_1_DIN -> Net-(J20-Pin_4)
Routing:
- net /24V_UNREGULATED: track 101.0 -> 48.2 mm
- net Net-(J9-Pin_4): track 0.00 -> 16.7 mm, vias 0 -> 1
- net Net-(J20-Pin_4): track 0.00 -> 16.4 mm, vias 0 -> 1
- net /ADC_1_CS: track 21.6 -> 8.09 mm, vias 1 -> 2
- net /ADC_2_CS: track 21.6 -> 8.10 mm, vias 1 -> 2
- net Net-(J9-Pin_6): track 0.00 -> 10.8 mm, vias 0 -> 1
- net Net-(J20-Pin_6): track 0.00 -> 10.3 mm, vias 0 -> 1
- net /ADC_1_DOUT: track 15.5 -> 7.47 mm, vias 1 -> 2
- net /ADC_2_DOUT: track 15.5 -> 7.52 mm, vias 1 -> 2
- net Net-(J9-Pin_1): track 0.00 -> 7.10 mm, vias 0 -> 1
- net Net-(J20-Pin_1): track 0.00 -> 6.85 mm, vias 0 -> 1
- net GND: track 53.9 -> 49.2 mm
- net /ADC_1_SCLK: track 11.8 -> 7.70 mm, vias 1 -> 2
- net Net-(J9-Pin_3): track 0.00 -> 4.10 mm, vias 0 -> 1
- net /ADC_2_SCLK: track 11.8 -> 7.72 mm, vias 1 -> 2
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- added copper zone on B.Cu, net /BATT_1
- removed copper zone on F.Cu, net /24V_REGULATED
- removed copper zone on F.Cu, net /5V_REGULATED

Commit message: updated LTC4372s, switch connector, ADC; added some power planes for other batteries
Parts:
- added C53: 22 nF, Capacitor_SMD:C_0201_0603Metric_Pad0.64x0.40mm_HandSolder, F.Cu at (275.4, 250.4)
- added RA15: 100, Resistor_SMD:R_0805_2012Metric_Pad1.20x1.40mm_HandSolder, F.Cu at (272.9, 250.5)
- moved R19 25.0 mm to (113.4, 110.6)
- moved R22 25.0 mm to (113.4, 135.6)
- moved R25 25.0 mm to (113.4, 160.6)
- moved R28 25.0 mm to (113.4, 185.6)
- moved RA14 2.29 mm to (272.9, 252.6)
- moved C29 2.26 mm to (267.4, 254.8)
- moved C31 2.26 mm to (273.1, 254.8)
- moved RA12 2.26 mm to (265.0, 254.8)
- moved RA13 2.26 mm to (269.8, 254.8)
- moved C30 2.26 mm to (272.3, 254.8)
- moved R35 0.97 mm to (280.6, 251.5)
- turned R12 to -90 degrees
- turned R15 to -90 degrees
- turned R18 to -90 degrees
- turned R21 to -90 degrees
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Connections:
- J18 pad 6: /5V_REG_SD -> unconnected-(J18-Pin_6-Pad6)
- Q12 pad 2: /BATT_IN_12_4 -> /BATT_IN_12_2
- Q14 pad 2: /BATT_IN_12_2 -> /BATT_IN_12_3
- Q16 pad 2: /BATT_IN_12_3 -> /BATT_IN_12_4
- Q18 pad 2: /BATT_IN_12_7 -> /BATT_IN_12_5
- Q20 pad 2: /BATT_IN_12_5 -> /BATT_IN_12_6
- Q22 pad 2: /BATT_IN_12_6 -> /BATT_IN_12_7
- U1 pad 7: unconnected-(U1-2UPU-Pad7) -> /SHDN
- U16 pad 11: unconnected-(U16-IN7-Pad11) -> Net-(U16-IN7)
- U2 pad 4: /BATT_IN_12_4 -> /BATT_IN_12_2
- U2 pad 7: unconnected-(U2-2UPU-Pad7) -> /SHDN
- U3 pad 4: /BATT_IN_12_2 -> /BATT_IN_12_3
- U3 pad 7: unconnected-(U3-2UPU-Pad7) -> /SHDN
- U4 pad 4: /BATT_IN_12_3 -> /BATT_IN_12_4
- U4 pad 7: unconnected-(U4-2UPU-Pad7) -> /SHDN
- U5 pad 4: /BATT_IN_12_7 -> /BATT_IN_12_5
- U5 pad 7: unconnected-(U5-2UPU-Pad7) -> /SHDN
- U6 pad 4: /BATT_IN_12_5 -> /BATT_IN_12_6
- U6 pad 7: unconnected-(U6-2UPU-Pad7) -> /SHDN
- U7 pad 4: /BATT_IN_12_6 -> /BATT_IN_12_7
- U7 pad 7: unconnected-(U7-2UPU-Pad7) -> /SHDN
Routing:
- net GND: track 49.2 -> 63.8 mm, vias 30 -> 43
- net /SHDN: track 1.40 -> 13.5 mm, vias 1 -> 7
- net Net-(U16-IN7): track 0.00 -> 9.80 mm
- net /THERM_8: track 0.00 -> 9.19 mm, vias 0 -> 1
- net Net-(D4-A): track 0.00 -> 7.41 mm
- net Net-(D7-A): track 0.00 -> 7.41 mm
- net Net-(D5-A): track 0.00 -> 7.41 mm
- net Net-(D3-A): track 0.00 -> 7.22 mm
- net Net-(D2-A): track 0.00 -> 7.22 mm
- net Net-(D8-A): track 0.00 -> 7.22 mm
- net Net-(D6-A): track 0.00 -> 7.22 mm
- net /THERM_7: track 1.94 -> 8.23 mm
- net Net-(U16-IN6): track 3.17 -> 7.19 mm
- net Net-(Q22-G): track 0.00 -> 3.78 mm
- net Net-(Q16-G): track 0.00 -> 3.78 mm
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- added copper zone on F.Cu, net /BATT_IN_12_2
- added copper zone on B.Cu, net Net-(J2-Pin_2)
- added copper zone on B.Cu, net Net-(J3-Pin_2)
- added copper zone on F.Cu, net Net-(J3-Pin_2)
- added copper zone on B.Cu, net Net-(J4-Pin_2)
- added copper zone on F.Cu, net Net-(J4-Pin_2)
- added copper zone on B.Cu, net Net-(J5-Pin_2)
- added copper zone on F.Cu, net Net-(J5-Pin_2)
- added copper zone on B.Cu, net Net-(J6-Pin_2)
- added copper zone on F.Cu, net Net-(J6-Pin_2)
- added copper zone on B.Cu, net Net-(J7-Pin_2)
- added copper zone on F.Cu, net Net-(J7-Pin_2)
- added copper zone on F.Cu, net Net-(Q11-S)
- added copper zone on B.Cu, net Net-(Q2-D)
- added copper zone on F.Cu, net Net-(Q2-D)
- added copper zone on B.Cu, net Net-(Q3-D)
- added copper zone on F.Cu, net Net-(Q3-D)
- added copper zone on B.Cu, net Net-(Q4-D)
- added copper zone on F.Cu, net Net-(Q4-D)
