File: Power Board 2/Power Board.kicad_pcb (KiCad board)
At the start: 4 copper layers, 187 parts, among them IC1 LTC4151IMS#PBF, IC2 LTC4151IMS#PBF, J1 Conn_01x02, J18 Conn_02x03_Top_Bottom, J19 Conn_01x02, J2 Conn_01x02, J21 Conn_01x02, J3 Conn_01x02, J4 Conn_01x02, J5 Conn_01x02, J6 Conn_01x02, J7 Conn_01x02, J8 Conn_01x02, J9 Conn_02x03_Top_Bottom, Q1 Q_PMOS_GDS, Q10 Q_NMOS_GDS, Q11 Q_NMOS_GDS, Q12 Q_NMOS_GDS, Q13 Q_NMOS_GDS, Q14 Q_NMOS_GDS, Q15 Q_NMOS_GDS, Q16 Q_NMOS_GDS, Q17 Q_NMOS_GDS, Q18 Q_NMOS_GDS, Q19 Q_NMOS_GDS, Q2 Q_PMOS_GDS, Q20 Q_NMOS_GDS, Q21 Q_NMOS_GDS, Q22 Q_NMOS_GDS, Q3 Q_PMOS_GDS, Q4 Q_PMOS_GDS, Q5 Q_PMOS_GDS, Q6 Q_PMOS_GDS, Q7 Q_PMOS_GDS, Q8 Q_PMOS_GDS, Q9 Q_NMOS_GDS, U1 LTC4372CDD-PBF, U10 ACS770xCB-050U-PFF, U11 ACS770xCB-050U-PFF, U12 ACS770xCB-050U-PFF, U13 ACS770xCB-050U-PFF, U14 ACS770xCB-050U-PFF, U15 ADC128S052CIMT, U17 TLV70033_SOT23-5, U2 LTC4372CDD-PBF, U3 LTC4372CDD-PBF, U4 LTC4372CDD-PBF, U5 LTC4372CDD-PBF, U6 LTC4372CDD-PBF, U7 LTC4372CDD-PBF, U8 ACS770xCB-050U-PFF, U9 ACS770xCB-050U-PFF

Commit message: changed mounting holes to without pad for star grounding
Parts:
- added H25: MountingHole_Pad, MountingHole:MountingHole_3.2mm_M3_DIN965, F.Cu at (149.5, 25.1)
- added H26: MountingHole_Pad, MountingHole:MountingHole_3.2mm_M3_DIN965, F.Cu at (197.8, 25.1)
- added H27: MountingHole_Pad, MountingHole:MountingHole_3.2mm_M3_DIN965, F.Cu at (198.8, 183.3)
- added H28: MountingHole_Pad, MountingHole:MountingHole_3.2mm_M3_DIN965, F.Cu at (198.8, 231.6)
- H1, H10, H2, H3, H4, H5, H6, H7, H8, H9: footprint MountingHole:MountingHole_3.2mm_M3_DIN965_Pad -> MountingHole:MountingHole_3.2mm_M3_DIN965
- moved J_I2C1 2.84 mm to (193.1, 229.5)
- moved J_I2C_Jetson1 0.81 mm to (193.1, 213.7)
- moved H5 0.18 mm to (52.8, 113.8)
- moved H10 0.15 mm to (101.1, 231.6)
- moved H7 0.15 mm to (52.8, 180.8)
- moved H8 0.15 mm to (101.1, 180.8)
- moved H9 0.15 mm to (52.8, 231.6)
Routing:
- net /SCL: track 47.8 -> 75.4 mm
- net /SDA: track 43.3 -> 54.5 mm
- net GND: vias 1350 -> 1349

Commit message: power board minor changes
Parts:
- C1, C10, C11, C12, C13, C14, C15, C16, C17, C18, C19, C2, C20, C21, C22, C23, C24, C3, C35, C36, C37, C38, C39, C4, C40, C41, C42, C43, C44, C45, C46, C47, C48, C49, C5, C50, C6, C7, C8, C9: footprint Capacitor_SMD:C_0201_0603Metric_Pad0.64x0.40mm_HandSolder -> Capacitor_SMD:C_0603_1608Metric
- C54: footprint Capacitor_SMD:C_0805_2012Metric_Pad1.18x1.45mm_HandSolder -> Capacitor_SMD:C_0805_2012Metric
- moved C1 1.62 mm to (116.3, 32.9)
- moved C24 1.56 mm to (184.3, 202.8)
- moved C3 1.55 mm to (116.3, 54.4)
- moved C9 1.50 mm to (116.3, 120.0)
- moved C5 1.41 mm to (116.3, 76.6)
- moved C13 1.41 mm to (116.3, 163.1)
- moved C21 1.34 mm to (174.0, 219.0)
- moved C49 1.33 mm to (168.8, 216.6)
- moved C17 1.30 mm to (176.6, 201.5)
- moved C23 1.25 mm to (182.3, 201.6)
- moved C11 1.23 mm to (116.3, 142.3)
- moved C50 1.08 mm to (171.3, 216.6)
- moved C22 0.88 mm to (179.6, 217.2)
- moved C7 0.88 mm to (116.3, 98.7)
- moved C46 0.87 mm to (159.8, 148.6)
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Routing:
- net GND: track 86.0 -> 68.4 mm, vias 1349 -> 1343
- net Net-(U15-IN2): track 8.45 -> 2.81 mm
- net /5V_REGULATED: track 37.2 -> 41.0 mm
- net /SHDN: track 166.4 -> 169.8 mm
- net /BATT_7_SENSE: track 63.9 -> 66.5 mm
- net GNDD: track 4.06 -> 2.10 mm
- net /3.3V: track 14.1 -> 15.9 mm
- net Net-(U15-IN1): track 6.74 -> 8.40 mm
- net /BATT_3_SENSE: track 132.2 -> 133.2 mm
- net /ADC_1_DOUT: track 7.47 -> 8.48 mm
- net Net-(C8-Pad1): track 3.43 -> 4.40 mm
- net Net-(U15-IN6): track 5.35 -> 6.31 mm
- net /BATT_1_SENSE: track 177.7 -> 178.6 mm
- net Net-(U15-IN5): track 5.31 -> 4.51 mm
- net /BATT_4_SENSE: track 110.1 -> 110.9 mm
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
Commit message: via stitching on power board
Routing:
- net Net-(Q21-S): vias 5 -> 45
- net Net-(Q19-S): vias 5 -> 44
- net Net-(Q17-S): vias 5 -> 45
- net Net-(Q15-S): vias 5 -> 45
- net Net-(Q13-S): vias 5 -> 42
- net Net-(Q11-S): vias 45 -> 48
- net /BATT_7_PRESENSE: vias 0 -> 105
- net /BATT_7: vias 220 -> 310
- net /BATT_6_PRESENSE: vias 0 -> 105
- net /BATT_6: vias 220 -> 310
- net /BATT_5_PRESENSE: vias 0 -> 105
- net /BATT_5: vias 220 -> 310
- net /BATT_4_PRESENSE: vias 0 -> 106
- net /BATT_4: vias 220 -> 310
- net /BATT_3_PRESENSE: vias 0 -> 105
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Other:
- board text added: "U9"
