File: Power Board 2/Power Board.kicad_sch (KiCad schematic)
At the start: 193 parts, among them IC1 LTC4151IMS#PBF, IC2 LTC4151IMS#PBF, J1 Conn_01x02, J18 Conn_02x03_Top_Bottom, J19 Conn_01x02, J2 Conn_01x02, J21 Conn_01x02, J3 Conn_01x02, J4 Conn_01x02, J5 Conn_01x02, J6 Conn_01x02, J7 Conn_01x02, J8 Conn_01x02, J9 Conn_02x03_Top_Bottom, Q1 Q_PMOS_GDS, Q10 Q_NMOS_GDS, Q11 Q_NMOS_GDS, Q12 Q_NMOS_GDS, Q13 Q_NMOS_GDS, Q14 Q_NMOS_GDS, Q15 Q_NMOS_GDS, Q16 Q_NMOS_GDS, Q17 Q_NMOS_GDS, Q18 Q_NMOS_GDS, Q19 Q_NMOS_GDS, Q2 Q_PMOS_GDS, Q20 Q_NMOS_GDS, Q21 Q_NMOS_GDS, Q22 Q_NMOS_GDS, Q3 Q_PMOS_GDS, Q4 Q_PMOS_GDS, Q5 Q_PMOS_GDS, Q6 Q_PMOS_GDS, Q7 Q_PMOS_GDS, Q8 Q_PMOS_GDS, Q9 Q_NMOS_GDS, U1 LTC4372CDD-PBF, U10 ACS770xCB-050U-PFF, U11 ACS770xCB-050U-PFF, U12 ACS770xCB-050U-PFF, U13 ACS770xCB-050U-PFF, U14 ACS770xCB-050U-PFF, U15 ADC128S052CIMT, U17 TLV70033_SOT23-5, U2 LTC4372CDD-PBF, U3 LTC4372CDD-PBF, U4 LTC4372CDD-PBF, U5 LTC4372CDD-PBF, U6 LTC4372CDD-PBF, U7 LTC4372CDD-PBF, U8 ACS770xCB-050U-PFF, U9 ACS770xCB-050U-PFF

Commit message: changed cap value in power board pcb according to datasheet calc
Parts:
- C15, C16, C17, C18, C19, C20, C21: value 22 nF -> 33 nF
Other:
- note added: "Implement shutdown before monitors, use power relay"
- note added: "VD also needs 1uf Cap I think (add it)"
