File: BMS Board/BMS Board.kicad_pcb (KiCad board)
At the start: 4 copper layers, 106.5 x 97 mm, 209 parts, among them J1 Conn_01x02, Q1 NMOS, U1 BQ76920PW, U10 TLV70033_SOT23-5, U2 TCA9548APWR, U3 BQ76920PW, U4 BQ76920PW, U5 BQ76920PW, U6 BQ76920PW, U7 BQ76920PW, U8 BQ76920PW, U9 BQ76930DBT

Commit message: used LDO output from BMs to Mux, routed PCB
Parts:
- C67, C68, C69, C70, C71, C72, C73, C74, C75, C76: value 220nF -> 1u
- R59, R60, R61, R62, R65, R66, R67, R68, R69: value 100 -> 1000
- U2: value TCA9548APWR -> t
- renumbered H4 to H1, H3 to H2, H5 to H3, H7 to H4, H2 to H5
Connections:
- C57 pad 2: Net-(U8-REGOUT) -> /MUX_PWR
- R71 pad 1: /3.3V -> /MUX_PWR
- R72 pad 1: /3.3V -> /MUX_PWR
- R73 pad 1: /3.3V -> /MUX_PWR
- R74 pad 1: /3.3V -> /MUX_PWR
- R75 pad 1: /3.3V -> /MUX_PWR
- R76 pad 1: /3.3V -> /MUX_PWR
- R77 pad 1: /3.3V -> /MUX_PWR
- R78 pad 1: /3.3V -> /MUX_PWR
- R87 pad 1: /3.3V -> /MUX_PWR
- U2 pad 24: /3.3V -> /MUX_PWR
- U8 pad 8: Net-(U8-REGOUT) -> /MUX_PWR
Routing:
- net /MUX_PWR: track 0.00 -> 90.6 mm, vias 0 -> 10
- net Net-(U8-REGOUT): track 4.19 -> 0.00 mm
- net /3.3V: track 3.68 -> 2.55 mm, vias 20 -> 10
- net /4S1-VC4: track 38.0 -> 38.8 mm
- net /4S3-VC4: track 38.0 -> 38.8 mm
- net /4S5-VC4: track 38.0 -> 38.6 mm
- net /4S7-VC4: track 38.0 -> 38.6 mm
- net /4S6-VC4: track 38.0 -> 38.6 mm
- net /4S4-VC4: track 38.0 -> 38.6 mm
- net /4S2-VC4: track 38.0 -> 38.6 mm
- net GND: vias 2677 -> 86
